File: kicad/cw.kicad_sch (KiCad schematic)
At the start: 110 parts, among them J1 AUDIO, J2 KEY, Q1 NPN, Q10 NPN, Q11 NPN, Q2 NMOS, Q3 NPN, Q4 NPN, Q6 NPN, Q7 NPN, Q8 NPN, Q9 NPN, SW1 TX/RX, SW2 TX/RX, SW3 FREQ_SELECT, U1 Si5351A-B-GT, U3 PCF8574TS, U4 RC1602A, Y1 4M, Y2 4M, Y3 4M, Y4 4M, Y5 4M, Y6 4M, Y7 4M, Y8 4M

Commit message: Update cw.kicad_sch
Parts:
- removed C35: 100n, symbol Device:C
- added Y10, Y11, Y12, Y13, Y14, Y15, Y9: 4M, symbol Device:Crystal
Connections:
- net at Q3.2 (B), R3.1, Y5.1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: now also Y13.1, Y14.1, Y15.1
- net at C1.1, C12.1, C16.1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: now also Y13.2, Y14.2, Y15.2
- net at Q1.3 (E), R22.1: now also L19.1
- net at J2.T, Y1.1, Y2.1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: now also Y10.1, Y11.1, Y12.1, Y9.1
- net at C9.1, Y1.2, Y2.2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: now also Y10.2, Y11.2, Y12.2, Y9.2; no longer C29.1
Other:
- moved on the sheet: C10, C11, C18, C19, C2, C20, C22, C3, C4, C6, C9, D2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

Commit message: Update cw.kicad_sch
Connections:
- net at C9.1, Y1.2, Y10.2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: now also C29.1
Other:
- moved on the sheet: C1, C20, C29, C9, L19, Q1, Q10, R15, R16, R19, R22, R4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

Commit message: Update cw.kicad_sch
Parts:
- added Y16: 4M, symbol Device:Crystal
Connections:
- net at Q3.2 (B), R3.1, Y13.1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: now also Y16.1
- net at C1.1, C12.1, C16.1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: now also Y16.2
- net at Y1.1, Y10.1, Y11.1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: now also J2.S; no longer J2.T
- net at C23.2, C41.2: now also J2.T; no longer J2.S
Other:
- moved on the sheet: AE1, C1, C10, C11, C12, C13, C14, C15, C16, C17, C18, C19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

Commit message: Update cw.kicad_sch
Connections:
- net +12V: no longer C21.2, C3.2, L12.2, L15.2, L20.1, L3.1, Q3.1 (C), Q6.1 (C)
- new net: C3.2, L15.2, L3.1, Q3.1 (C)
- new net: C21.2, L12.2, L20.1, Q6.1 (C)
Other:
- moved on the sheet: A1, AE1, BT1, C1, C10, C11, C12, C13, C14, C15, C16, C17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

Commit message: Update cw.kicad_sch
Parts:
- removed C41: 10p, symbol Device:C
- added C26: 10p, symbol Device:C
Connections:
- net at C23.2, J2.T: now also C26.2
- net at C23.1, L1.2: now also C26.1
Changed lines of the file:
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@@
-    )
-  )
-  (symbol (lib_id "Device:C") (at 266.7 242.57 90) (unit 1)
-    (in_bom yes) (on_board yes) (dnp no) (fields_autoplaced)
-    (property "Reference" "C41" (at 266.7 234.95 90)
-      (effects (font (size 1.27 1.27)) hide)
-    )
-    (property "Value" "10p" (at 266.7 237.49 90)
-      (effects (font (size 1.27 1.27)))
-    )
-    (property "Footprint" "" (at 270.51 241.6048 0)
-      (effects (font (size 1.27 1.27)) hide)
-    )
-    (property "Datasheet" "~" (at 266.7 242.57 0)
-      (effects (font (size 1.27 1.27)) hide)
-    )
-    (pin "1")
-    (pin "2")
-    (instances
-      (project "cw"
-        (path "/817248d0-f027-4dd0-8ccd-515a582be88c"
-          (reference "C41") (unit 1)
-        )
-      )
     )
   )
@@
         )
       )
+    )
+  )
+  (symbol (lib_id "Device:C") (at 266.7 242.57 90) (unit 1)
+    (in_bom yes) (on_board yes) (dnp no) (fields_autoplaced)
+    (property "Reference" "C26" (at 266.7 234.95 90)
+      (effects (font (size 1.27 1.27)))
+    )
+    (property "Value" "10p" (at 266.7 237.49 90)
+      (effects (font (size 1.27 1.27)))
+    )
+    (property "Footprint" "" (at 270.51 241.6048 0)
+      (effects (font (size 1.27 1.27)) hide)
+    )
+    (property "Datasheet" "~" (at 266.7 242.57 0)
+      (effects (font (size 1.27 1.27)) hide)
+    )
+    (pin "1")
+    (pin "2")
+    (instances
+      (project "cw"
+        (path "/817248d0-f027-4dd0-8ccd-515a582be88c"
+          (reference "C26") (unit 1)
+        )
+      )

Commit message: Update cw.kicad_sch
Parts:
- added C30, C32, C34, C36: 220p, symbol Device:C
- added C31, C33, C35, C37, C39, C41, C49, C51: 10p, symbol Device:C
- added C38, C40, C44, C50: 33p, symbol Device:C
- added L16, L18, L21, L22: 6u8, symbol Device:L
- added L23, L24, L25, L26: 4u7, symbol Device:L
Connections:
- net GND: now also C30.1, C31.1, C32.1, C33.1, C34.1, C35.1, C36.1, C37.1, C38.1, C39.1, C40.1, C41.1, C44.1, C49.1, C50.1, C51.1, L16.1, L18.1, L21.1, L22.1, L23.1, L24.1, L25.1, L26.1
- net at L11.1, Q9.3 (E), R14.1: now also C44.2, C49.2, L25.2
- net at C11.1, C20.2, C43.2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: now also C40.2, C41.2, L24.2
- net at C19.2, C2.1, C22.1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: now also C36.2, C37.2, L22.2
- net at C15.2, C17.1, C47.2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: now also C50.2, C51.2, L26.2
- net at L1.1, Q11.3 (E), R12.1: now also C30.2, C31.2, L16.2
- net at C23.2, C26.2, J2.T: now also C32.2, C33.2, L18.2
- net at L9.1, Q7.3 (E), R8.1: now also C38.2, C39.2, L23.2
- net at L7.1, Q8.3 (E), R13.1: now also C34.2, C35.2, L21.2
Other:
- moved on the sheet: A1, AE1, BT1, C1, C10, C11, C12, C13, C14, C15, C16, C17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
